Commit message: readme update

File: ardupilot_sitl_gazebo_plugin/urdf/recorder_camera.xacro (robot description, xacro)
@@ -5,5 +5,5 @@
   xmlns:xacro="http://ros.org/wiki/xacro"
   >
-    <property name="M_PI" value="3.1415926535897931" />
+    <xacro:property name="M_PI" value="3.1415926535897931" />
   <xacro:macro name="recorder_camera" params="name parent *origin ros_topic update_rate res_x res_y image_format hfov video_dir video_filename video_fileext">
       <joint name="${name}_joint" type="fixed">

File: ardupilot_sitl_gazebo_plugin/urdf/sensors/generic_camera.urdf.xacro (robot description, xacro)
@@ -5,5 +5,5 @@
   xmlns:xacro="http://ros.org/wiki/xacro"
   >
-    <property name="M_PI" value="3.1415926535897931" />
+    <xacro:property name="M_PI" value="3.1415926535897931" />
   <xacro:macro name="generic_camera" params="name parent *origin ros_topic cam_info_topic update_rate res_x res_y image_format hfov framename">
     <joint name="${name}_joint" type="fixed">

File: ardupilot_sitl_gazebo_plugin/urdf/sensors/kinect.urdf.xacro (robot description, xacro)
@@ -1,10 +1,10 @@
 <?xml version="1.0"?>
 <robot name="sensor_kinect" xmlns:xacro="http://ros.org/wiki/xacro">
-  <property name="cam_px" value="1.63" />
+  <xacro:property name="cam_px" value="1.63" />
   <xacro:property name="kinect_cam_py" value="-0.0125"/>
-  <property name="cam_pz" value="0.68" />
-  <property name="cam_or" value="0" />
-  <property name="cam_op" value="0" />
-  <property name="cam_oy" value="0" />
+  <xacro:property name="cam_pz" value="0.68" />
+  <xacro:property name="cam_or" value="0" />
+  <xacro:property name="cam_op" value="0" />
+  <xacro:property name="cam_oy" value="0" />
   <xacro:property name="M_PI" value="3.1415926535897931" />
   <!-- Parameterised in part by the values in turtlebot_properties.urdf.xacro -->
